Commit message: can walk, but unstable

File: bipedal_robot_description/h1_description/urdf/h1_with_sole.urdf (robot description, URDF)
Before this commit: robot h1_description, 27 links, 26 joints
Links:
- removed link left_sole_link
- removed link right_sole_link
- added link left_sole_1_link, mass 0.01; collision sphere radius=0.001; visual sphere radius=0.001
- added link left_sole_2_link, mass 0.01; collision sphere radius=0.001; visual sphere radius=0.001
- added link right_sole_1_link, mass 0.01; collision sphere radius=0.001; visual sphere radius=0.001
- added link right_sole_2_link, mass 0.01; collision sphere radius=0.001; visual sphere radius=0.001
Joints:
- removed joint left_sole_joint
- removed joint right_sole_joint
- added joint left_sole_1_joint: type fixed, parent left_ankle_link, child left_sole_1_link, origin xyz=0.19 0.0 -0.06 rpy=0 0 0
- added joint left_sole_2_joint: type fixed, parent left_ankle_link, child left_sole_2_link, origin xyz=-0.1 0.0 -0.06 rpy=0 0 0
- added joint right_sole_1_joint: type fixed, parent right_ankle_link, child right_sole_1_link, origin xyz=0.19 0.0 -0.06 rpy=0 0 0
- added joint right_sole_2_joint: type fixed, parent right_ankle_link, child right_sole_2_link, origin xyz=-0.1 0.0 -0.06 rpy=0 0 0
