Commit message: add support for h1

File: bipedal_robot_example/unitree_h1/h1_description/urdf/h1.urdf (robot description, URDF)
Before this commit: robot h1_description, 25 links, 24 joints
Joints:
- joint left_hip_pitch_joint: limit lower=-3.14 upper=2.53 effort=200 velocity=23 -> lower=-1.57 upper=1.57 effort=200 velocity=23
- joint right_hip_pitch_joint: limit lower=-3.14 upper=2.53 effort=200 velocity=23 -> lower=-1.57 upper=1.57 effort=200 velocity=23

File: bipedal_robot_example/unitree_h1/h1_description/urdf/h1_gazebo.urdf (robot description, URDF)
Before this commit: robot h1_description, 29 links, 28 joints
Links:
- removed link left_sole_1_link
- removed link left_sole_2_link
- removed link right_sole_1_link
- removed link right_sole_2_link
- link imu_link: mass None -> 0.01
Joints:
- removed joint left_sole_1_joint
- removed joint left_sole_2_joint
- removed joint right_sole_1_joint
- removed joint right_sole_2_joint
- joint left_hip_pitch_joint: limit lower=-3.14 upper=2.53 effort=200 velocity=23 -> lower=-1.57 upper=1.57 effort=200 velocity=23
- joint right_hip_pitch_joint: limit lower=-3.14 upper=2.53 effort=200 velocity=23 -> lower=-1.57 upper=1.57 effort=200 velocity=23

File: bipedal_robot_example/unitree_h1/h1_description/urdf/h1_with_sole.urdf (robot description, URDF)
Before this commit: robot h1_description, 29 links, 28 joints
Joints:
- joint left_hip_pitch_joint: limit lower=-3.14 upper=2.53 effort=200 velocity=23 -> lower=-1.57 upper=1.57 effort=200 velocity=23
- joint right_hip_pitch_joint: limit lower=-3.14 upper=2.53 effort=200 velocity=23 -> lower=-1.57 upper=1.57 effort=200 velocity=23

Commit message: h1 walk

File: bipedal_robot_example/unitree_h1/h1_description/urdf/h1.urdf (robot description, URDF)
Before this commit: robot h1_description, 25 links, 24 joints
Joints:
- joint torso_joint: limit lower=-2.35 upper=2.35 effort=200 velocity=23 -> lower=-1.0 upper=1.0 effort=200 velocity=23

File: bipedal_robot_example/unitree_h1/h1_description/urdf/h1_gazebo.urdf (robot description, URDF)
Before this commit: robot h1_description, 25 links, 24 joints
Joints:
- joint torso_joint: limit lower=-2.35 upper=2.35 effort=200 velocity=23 -> lower=-1.0 upper=1.0 effort=200 velocity=23

File: bipedal_robot_example/unitree_h1/h1_description/urdf/h1_with_sole.urdf (robot description, URDF)
Before this commit: robot h1_description, 29 links, 28 joints
Joints:
- joint torso_joint: limit lower=-2.35 upper=2.35 effort=200 velocity=23 -> lower=-1.0 upper=1.0 effort=200 velocity=23
