Commit message: bak

File: bipedal_robot_example/openloong_description/urdf/AzureLoong_gazebo.urdf (robot description, URDF)
Before this commit: robot OpenLoong, 33 links, 32 joints
Links:
- link Link_ankle_l_pitch: geometry collision box size=0.02199999988079071 0.02199999988079071 0.0608999989926815; visual mesh filename=package://openloong_description/meshes/Link_ankle_l_pitch.S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
- link Link_ankle_l_roll: geometry collision box size=0.08042679535932826 0.08830404889775641 0.24500000476837158; visual mesh filename=package://openloong_description/meshes/Link_ankle_l_roll.STL
- link Link_ankle_r_pitch: geometry collision box size=0.02199999988079071 0.02199999988079071 0.0608999989926815; visual mesh filename=package://openloong_description/meshes/Link_ankle_r_pitch.S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
- link Link_ankle_r_roll: geometry collision box size=0.08003152899406105 0.08708268283896033 0.2450051728352756; visual mesh filename=package://openloong_description/meshes/Link_ankle_r_roll.STL
- link Link_arm_l_01: geometry collision box size=0.07599999755620956 0.0835999995470047 0.08499999437481165; visual mesh filename=package://openloong_description/meshes/Link_arm_l_01.STL
- link Link_arm_l_02: geometry collision box size=0.07599999755620956 0.10800000187009573 0.1523812673985958; visual mesh filename=package://openloong_description/meshes/Link_arm_l_02.STL
- link Link_arm_l_03: geometry collision box size=0.07793724111544645 0.08272916659551086 0.22364142748542543; visual mesh filename=package://openloong_description/meshes/Link_arm_l_03.STL
- link Link_arm_l_04: geometry collision box size=0.0700463031850532 0.09969999734312296 0.14310730744646838; visual mesh filename=package://openloong_description/meshes/Link_arm_l_04.STL
- link Link_arm_l_05: geometry collision box size=0.060499999672174454 0.0949999988079071 0.2250000089644455; visual mesh filename=package://openloong_description/meshes/Link_arm_l_05.STL
- link Link_arm_l_06: geometry collision sphere radius=0.03501915449457261; visual mesh filename=package://openloong_description/meshes/Link_arm_l_06.STL
- link Link_arm_l_07: geometry collision box size=0.07420478960456942 0.14182928051113333 0.3122642579482233; visual mesh filename=package://openloong_description/meshes/Link_arm_l_07.STL
- link Link_arm_r_01: geometry collision box size=0.07599999755620956 0.0835999995470047 0.08499999437481165; visual mesh filename=package://openloong_description/meshes/Link_arm_r_01.STL
- link Link_arm_r_02: geometry collision box size=0.07599999755620956 0.10800000187009573 0.1523812673985958; visual mesh filename=package://openloong_description/meshes/Link_arm_r_02.STL
- link Link_arm_r_03: geometry collision box size=0.07793724111544645 0.08272916659551086 0.22364142748542531; visual mesh filename=package://openloong_description/meshes/Link_arm_r_03.STL
- link Link_arm_r_04: geometry collision box size=0.0700463031850532 0.09969999734312296 0.14310730744646838; visual mesh filename=package://openloong_description/meshes/Link_arm_r_04.STL
- link Link_arm_r_05: geometry collision box size=0.060499999672174454 0.0949999988079071 0.22500000896444527; visual mesh filename=package://openloong_description/meshes/Link_arm_r_05.STL
- link Link_arm_r_06: geometry collision sphere radius=0.035019154494572595; visual mesh filename=package://openloong_description/meshes/Link_arm_r_06.STL
- link Link_arm_r_07: geometry collision box size=0.07446015413122065 0.14150577388908692 0.3121386277707064; visual mesh filename=package://openloong_description/meshes/Link_arm_r_07.STL
- link Link_head_pitch: geometry collision cylinder length=0.24085526634007692 radius=0.09356938956827072; visual mesh filename=package://openloong_description/meshes/Link_head_pitch.STL
- link Link_head_yaw: geometry collision box size=0.06460000015795231 0.07999999821186066 0.09130000043660402; visual mesh filename=package://openloong_description/meshes/Link_head_yaw.STL
- link Link_hip_l_pitch: geometry collision box size=0.1286939637515551 0.15699999779462814 0.47319313536392066; visual mesh filename=package://openloong_description/meshes/Link_hip_l_pitch.STL
- link Link_hip_l_roll: geometry collision box size=0.10953407117352178 0.11355194626876655 0.14642735745762184; visual mesh filename=package://openloong_description/meshes/Link_hip_l_roll.STL
- link Link_hip_l_yaw: geometry collision box size=0.13824999704957008 0.15199876576662064 0.16399998776614666; visual mesh filename=package://openloong_description/meshes/Link_hip_l_yaw.STL
- link Link_hip_r_pitch: geometry collision box size=0.12843006439604737 0.15761262328366868 0.47204802623524966; visual mesh filename=package://openloong_description/meshes/Link_hip_r_pitch.STL
- link Link_hip_r_roll: geometry collision box size=0.10938711969958106 0.11348148586759206 0.1466289123198961; visual mesh filename=package://openloong_description/meshes/Link_hip_r_roll.STL
- link Link_hip_r_yaw: geometry collision box size=0.13824999704957008 0.15199876576662064 0.16399998776614666; visual mesh filename=package://openloong_description/meshes/Link_hip_r_yaw.STL
- link Link_knee_l_pitch: geometry collision box size=0.0830744339109904 0.10167547683539807 0.470009645389421; visual mesh filename=package://openloong_description/meshes/Link_knee_l_pitch.STL
- link Link_knee_r_pitch: geometry collision box size=0.08305011195946374 0.10171538619274088 0.4700031674581286; visual mesh filename=package://openloong_description/meshes/Link_knee_r_pitch.STL
- link Link_waist_pitch: geometry collision box size=0.11948809772729874 0.14000000804662704 0.14300000621005893; visual mesh filename=package://openloong_description/meshes/Link_waist_pitch.STL
- link Link_waist_roll: geometry collision box size=0.11984597891569138 0.15949999913573265 0.23099999874830246; visual mesh filename=package://openloong_description/meshes/Link_waist_roll.STL
- link Link_waist_yaw: geometry collision box size=0.13895585224963725 0.24769999831914902 0.37378689646720886; visual mesh filename=package://openloong_description/meshes/Link_waist_yaw.STL
- link base_link: geometry collision box size=0.3273754417896271 0.36503949132581104 0.42854637797201894; visual mesh filename=package://openloong_description/meshes/base_link.STL

File: bipedal_robot_example/openloong_description/urdf/AzureLoong_simplified.urdf (robot description, URDF)
Before this commit: robot OpenLoog, 32 links, 31 joints
Links:
- link Link_ankle_l_pitch: geometry collision box size=0.02199999988079071 0.02199999988079071 0.0608999989926815; visual mesh filename=package://openloong_description/meshes/Link_ankle_l_pitch.S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
- link Link_ankle_l_roll: geometry collision box size=0.08042679535932826 0.08830404889775641 0.24500000476837158; visual mesh filename=package://openloong_description/meshes/Link_ankle_l_roll.STL
- link Link_ankle_r_pitch: geometry collision box size=0.02199999988079071 0.02199999988079071 0.0608999989926815; visual mesh filename=package://openloong_description/meshes/Link_ankle_r_pitch.S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
- link Link_ankle_r_roll: geometry collision box size=0.08003152899406105 0.08708268283896033 0.2450051728352756; visual mesh filename=package://openloong_description/meshes/Link_ankle_r_roll.STL
- link Link_arm_l_01: geometry collision box size=0.07599999755620956 0.0835999995470047 0.08499999437481165; visual mesh filename=package://openloong_description/meshes/Link_arm_l_01.STL
- link Link_arm_l_02: geometry collision box size=0.07599999755620956 0.10800000187009573 0.1523812673985958; visual mesh filename=package://openloong_description/meshes/Link_arm_l_02.STL
- link Link_arm_l_03: geometry collision box size=0.07793724111544645 0.08272916659551086 0.22364142748542543; visual mesh filename=package://openloong_description/meshes/Link_arm_l_03.STL
- link Link_arm_l_04: geometry collision box size=0.0700463031850532 0.09969999734312296 0.14310730744646838; visual mesh filename=package://openloong_description/meshes/Link_arm_l_04.STL
- link Link_arm_l_05: geometry collision box size=0.060499999672174454 0.0949999988079071 0.2250000089644455; visual mesh filename=package://openloong_description/meshes/Link_arm_l_05.STL
- link Link_arm_l_06: geometry collision sphere radius=0.03501915449457261; visual mesh filename=package://openloong_description/meshes/Link_arm_l_06.STL
- link Link_arm_l_07: geometry collision box size=0.07420478960456942 0.14182928051113333 0.3122642579482233; visual mesh filename=package://openloong_description/meshes/Link_arm_l_07.STL
- link Link_arm_r_01: geometry collision box size=0.07599999755620956 0.0835999995470047 0.08499999437481165; visual mesh filename=package://openloong_description/meshes/Link_arm_r_01.STL
- link Link_arm_r_02: geometry collision box size=0.07599999755620956 0.10800000187009573 0.1523812673985958; visual mesh filename=package://openloong_description/meshes/Link_arm_r_02.STL
- link Link_arm_r_03: geometry collision box size=0.07793724111544645 0.08272916659551086 0.22364142748542531; visual mesh filename=package://openloong_description/meshes/Link_arm_r_03.STL
- link Link_arm_r_04: geometry collision box size=0.0700463031850532 0.09969999734312296 0.14310730744646838; visual mesh filename=package://openloong_description/meshes/Link_arm_r_04.STL
- link Link_arm_r_05: geometry collision box size=0.060499999672174454 0.0949999988079071 0.22500000896444527; visual mesh filename=package://openloong_description/meshes/Link_arm_r_05.STL
- link Link_arm_r_06: geometry collision sphere radius=0.035019154494572595; visual mesh filename=package://openloong_description/meshes/Link_arm_r_06.STL
- link Link_arm_r_07: geometry collision box size=0.07446015413122065 0.14150577388908692 0.3121386277707064; visual mesh filename=package://openloong_description/meshes/Link_arm_r_07.STL
- link Link_head_pitch: geometry collision cylinder length=0.24085526634007692 radius=0.09356938956827072; visual mesh filename=package://openloong_description/meshes/Link_head_pitch.STL
- link Link_head_yaw: geometry collision box size=0.06460000015795231 0.07999999821186066 0.09130000043660402; visual mesh filename=package://openloong_description/meshes/Link_head_yaw.STL
- link Link_hip_l_pitch: geometry collision box size=0.1286939637515551 0.15699999779462814 0.47319313536392066; visual mesh filename=package://openloong_description/meshes/Link_hip_l_pitch.STL
- link Link_hip_l_roll: geometry collision box size=0.10953407117352178 0.11355194626876655 0.14642735745762184; visual mesh filename=package://openloong_description/meshes/Link_hip_l_roll.STL
- link Link_hip_l_yaw: geometry collision box size=0.13824999704957008 0.15199876576662064 0.16399998776614666; visual mesh filename=package://openloong_description/meshes/Link_hip_l_yaw.STL
- link Link_hip_r_pitch: geometry collision box size=0.12843006439604737 0.15761262328366868 0.47204802623524966; visual mesh filename=package://openloong_description/meshes/Link_hip_r_pitch.STL
- link Link_hip_r_roll: geometry collision box size=0.10938711969958106 0.11348148586759206 0.1466289123198961; visual mesh filename=package://openloong_description/meshes/Link_hip_r_roll.STL
- link Link_hip_r_yaw: geometry collision box size=0.13824999704957008 0.15199876576662064 0.16399998776614666; visual mesh filename=package://openloong_description/meshes/Link_hip_r_yaw.STL
- link Link_knee_l_pitch: geometry collision box size=0.0830744339109904 0.10167547683539807 0.470009645389421; visual mesh filename=package://openloong_description/meshes/Link_knee_l_pitch.STL
- link Link_knee_r_pitch: geometry collision box size=0.08305011195946374 0.10171538619274088 0.4700031674581286; visual mesh filename=package://openloong_description/meshes/Link_knee_r_pitch.STL
- link Link_waist_pitch: geometry collision box size=0.11948809772729874 0.14000000804662704 0.14300000621005893; visual mesh filename=package://openloong_description/meshes/Link_waist_pitch.STL
- link Link_waist_roll: geometry collision box size=0.11984597891569138 0.15949999913573265 0.23099999874830246; visual mesh filename=package://openloong_description/meshes/Link_waist_roll.STL
- link Link_waist_yaw: geometry collision box size=0.13895585224963725 0.24769999831914902 0.37378689646720886; visual mesh filename=package://openloong_description/meshes/Link_waist_yaw.STL
- link base_link: geometry collision box size=0.3273754417896271 0.36503949132581104 0.42854637797201894; visual mesh filename=package://openloong_description/meshes/base_link.STL

File: bipedal_robot_example/openloong_description/urdf/AzureLoong_with_sole.urdf (robot description, URDF)
Before this commit: robot OpenLoong, 36 links, 35 joints
Links:
- link Link_ankle_l_pitch: geometry collision box size=0.02199999988079071 0.02199999988079071 0.0608999989926815; visual mesh filename=package://openloong_description/meshes/Link_ankle_l_pitch.S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
- link Link_ankle_l_roll: geometry collision box size=0.08042679535932826 0.08830404889775641 0.24500000476837158; visual mesh filename=package://openloong_description/meshes/Link_ankle_l_roll.STL
- link Link_ankle_r_pitch: geometry collision box size=0.02199999988079071 0.02199999988079071 0.0608999989926815; visual mesh filename=package://openloong_description/meshes/Link_ankle_r_pitch.S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
- link Link_ankle_r_roll: geometry collision box size=0.08003152899406105 0.08708268283896033 0.2450051728352756; visual mesh filename=package://openloong_description/meshes/Link_ankle_r_roll.STL
- link Link_arm_l_01: geometry collision box size=0.07599999755620956 0.0835999995470047 0.08499999437481165; visual mesh filename=package://openloong_description/meshes/Link_arm_l_01.STL
- link Link_arm_l_02: geometry collision box size=0.07599999755620956 0.10800000187009573 0.1523812673985958; visual mesh filename=package://openloong_description/meshes/Link_arm_l_02.STL
- link Link_arm_l_03: geometry collision box size=0.07793724111544645 0.08272916659551086 0.22364142748542543; visual mesh filename=package://openloong_description/meshes/Link_arm_l_03.STL
- link Link_arm_l_04: geometry collision box size=0.0700463031850532 0.09969999734312296 0.14310730744646838; visual mesh filename=package://openloong_description/meshes/Link_arm_l_04.STL
- link Link_arm_l_05: geometry collision box size=0.060499999672174454 0.0949999988079071 0.2250000089644455; visual mesh filename=package://openloong_description/meshes/Link_arm_l_05.STL
- link Link_arm_l_06: geometry collision sphere radius=0.03501915449457261; visual mesh filename=package://openloong_description/meshes/Link_arm_l_06.STL
- link Link_arm_l_07: geometry collision box size=0.07420478960456942 0.14182928051113333 0.3122642579482233; visual mesh filename=package://openloong_description/meshes/Link_arm_l_07.STL
- link Link_arm_r_01: geometry collision box size=0.07599999755620956 0.0835999995470047 0.08499999437481165; visual mesh filename=package://openloong_description/meshes/Link_arm_r_01.STL
- link Link_arm_r_02: geometry collision box size=0.07599999755620956 0.10800000187009573 0.1523812673985958; visual mesh filename=package://openloong_description/meshes/Link_arm_r_02.STL
- link Link_arm_r_03: geometry collision box size=0.07793724111544645 0.08272916659551086 0.22364142748542531; visual mesh filename=package://openloong_description/meshes/Link_arm_r_03.STL
- link Link_arm_r_04: geometry collision box size=0.0700463031850532 0.09969999734312296 0.14310730744646838; visual mesh filename=package://openloong_description/meshes/Link_arm_r_04.STL
- link Link_arm_r_05: geometry collision box size=0.060499999672174454 0.0949999988079071 0.22500000896444527; visual mesh filename=package://openloong_description/meshes/Link_arm_r_05.STL
- link Link_arm_r_06: geometry collision sphere radius=0.035019154494572595; visual mesh filename=package://openloong_description/meshes/Link_arm_r_06.STL
- link Link_arm_r_07: geometry collision box size=0.07446015413122065 0.14150577388908692 0.3121386277707064; visual mesh filename=package://openloong_description/meshes/Link_arm_r_07.STL
- link Link_head_pitch: geometry collision cylinder length=0.24085526634007692 radius=0.09356938956827072; visual mesh filename=package://openloong_description/meshes/Link_head_pitch.STL
- link Link_head_yaw: geometry collision box size=0.06460000015795231 0.07999999821186066 0.09130000043660402; visual mesh filename=package://openloong_description/meshes/Link_head_yaw.STL
- link Link_hip_l_pitch: geometry collision box size=0.1286939637515551 0.15699999779462814 0.47319313536392066; visual mesh filename=package://openloong_description/meshes/Link_hip_l_pitch.STL
- link Link_hip_l_roll: geometry collision box size=0.10953407117352178 0.11355194626876655 0.14642735745762184; visual mesh filename=package://openloong_description/meshes/Link_hip_l_roll.STL
- link Link_hip_l_yaw: geometry collision box size=0.13824999704957008 0.15199876576662064 0.16399998776614666; visual mesh filename=package://openloong_description/meshes/Link_hip_l_yaw.STL
- link Link_hip_r_pitch: geometry collision box size=0.12843006439604737 0.15761262328366868 0.47204802623524966; visual mesh filename=package://openloong_description/meshes/Link_hip_r_pitch.STL
- link Link_hip_r_roll: geometry collision box size=0.10938711969958106 0.11348148586759206 0.1466289123198961; visual mesh filename=package://openloong_description/meshes/Link_hip_r_roll.STL
- link Link_hip_r_yaw: geometry collision box size=0.13824999704957008 0.15199876576662064 0.16399998776614666; visual mesh filename=package://openloong_description/meshes/Link_hip_r_yaw.STL
- link Link_knee_l_pitch: geometry collision box size=0.0830744339109904 0.10167547683539807 0.470009645389421; visual mesh filename=package://openloong_description/meshes/Link_knee_l_pitch.STL
- link Link_knee_r_pitch: geometry collision box size=0.08305011195946374 0.10171538619274088 0.4700031674581286; visual mesh filename=package://openloong_description/meshes/Link_knee_r_pitch.STL
- link Link_waist_pitch: geometry collision box size=0.11948809772729874 0.14000000804662704 0.14300000621005893; visual mesh filename=package://openloong_description/meshes/Link_waist_pitch.STL
- link Link_waist_roll: geometry collision box size=0.11984597891569138 0.15949999913573265 0.23099999874830246; visual mesh filename=package://openloong_description/meshes/Link_waist_roll.STL
- link Link_waist_yaw: geometry collision box size=0.13895585224963725 0.24769999831914902 0.37378689646720886; visual mesh filename=package://openloong_description/meshes/Link_waist_yaw.STL
- link base_link: geometry collision box size=0.3273754417896271 0.36503949132581104 0.42854637797201894; visual mesh filename=package://openloong_description/meshes/base_link.STL
